File: kicad/PMM-1.0-R1.kicad_sch (KiCad schematic)
At the start: 2 parts, among them U3 STM32C031C4T6

Commit message: update gitignore and whatnot
Parts:
- renumbered C27 to C1, U3 to U1
Changed lines of the file:
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@@
 	(paper "A4")
+	(junction
+		(at 100.33 27.94)
+		(diameter 0)
+		(color 0 0 0 0)
+	)
 	(junction
 		(at 204.47 17.78)
@@
 	(wire
 		(pts
-			(xy 35.56 48.26) (xy 36.83 48.26)
-		)
-		(stroke
-			(width 0)
-			(type default)
-		)
-	)
-	(wire
-		(pts
-			(xy 90.17 54.61) (xy 92.71 54.61)
+			(xy 36.83 27.94) (xy 38.1 27.94)
+		)
+		(stroke
+			(width 0)
+			(type default)
+		)
+	)
+	(wire
+		(pts
+			(xy 99.06 59.69) (xy 101.6 59.69)
 		)
 		(stroke
@@
 	(wire
 		(pts
-			(xy 35.56 50.8) (xy 36.83 50.8)
+			(xy 63.5 27.94) (xy 76.2 27.94)
+		)
+		(stroke
+			(width 0)
+			(type default)
+		)
+	)
+	(wire
+		(pts
+			(xy 36.83 30.48) (xy 38.1 30.48)
+		)
+		(stroke
+			(width 0)
+			(type default)
+		)
+	)
+	(wire
+		(pts
+			(xy 100.33 53.34) (xy 101.6 53.34)
 		)
 		(stroke
@@
 	(wire
 		(pts
+			(xy 100.33 27.94) (xy 100.33 53.34)
+		)
+		(stroke
+			(width 0)
+			(type default)
+		)
+	)
+	(wire
+		(pts
+			(xy 101.6 27.94) (xy 100.33 27.94)
+		)
+		(stroke
+			(width 0)
+			(type default)
+		)
+	)
+	(wire
+		(pts
 			(xy 204.47 17.78) (xy 204.47 19.05)
 		)
@@
 	(wire
 		(pts
-			(xy 80.01 48.26) (xy 92.71 48.26)
+			(xy 88.9 27.94) (xy 100.33 27.94)
 		)
 		(stroke
@@
 	(wire
 		(pts
-			(xy 35.56 53.34) (xy 36.83 53.34)
+			(xy 36.83 33.02) (xy 38.1 33.02)
 		)
 		(stroke
@@
 	(global_label "GPOUT"
 		(shape input)
-		(at 35.56 48.26 180)
+		(at 36.83 27.94 180)
 		(fields_autoplaced yes)
 		(effects
@@
 		)
 		(property "Intersheetrefs" "${INTERSHEET_REFS}"
-			(at 26.4062 48.26 0)
+			(at 27.6762 27.94 0)
 			(hide yes)
 			(show_name no)
@@
 	(global_label "PACK+"
 		(shape input)
-		(at 35.56 50.8 180)
+		(at 36.83 30.48 180)
 		(fields_autoplaced yes)
 		(effects
@@
 		)
 		(property "Intersheetrefs" "${INTERSHEET_REFS}"
-			(at 26.1038 50.8 0)
+			(at 27.3738 30.48 0)
 			(hide yes)
 			(show_name no)
@@
 	(global_label "TPS2291_ON"
 		(shape input)
-		(at 90.17 54.61 180)
+		(at 99.06 59.69 180)
 		(fields_autoplaced yes)
 		(effects
@@
 		)
 		(property "Intersheetrefs" "${INTERSHEET_REFS}"
-			(at 75.2711 54.61 0)
+			(at 84.1611 59.69 0)
 			(hide yes)
 			(show_name no)
@@
 	(global_label "PACK-"
 		(shape input)
-		(at 35.56 53.34 180)
+		(at 36.83 33.02 180)
 		(fields_autoplaced yes)
 		(effects
@@
 		)
 		(property "Intersheetrefs" "${INTERSHEET_REFS}"
-			(at 26.1038 53.34 0)
+			(at 27.3738 33.02 0)
 			(hide yes)
 			(show_name no)
@@
 		(dnp no)
 		(fields_autoplaced yes)
-		(property "Reference" "C27"
+		(property "Reference" "C1"
 			(at 207.01 20.3262 0)
 			(show_name no)
@@
 			(project "PMM-1.0-R1"
 				(path "/dfbd1ee6-4059-4519-bc2e-4814be9dda35"
-					(reference "C27")
+					(reference "C1")
 					(unit 1)
 				)
@@
 		(dnp no)
 		(fields_autoplaced yes)
-		(property "Reference" "#PWR017"
+		(property "Reference" "#PWR03"
 			(at 233.68 125.73 0)
 			(hide yes)
@@
 			(project "PMM-1.0-R1"
 				(path "/dfbd1ee6-4059-4519-bc2e-4814be9dda35"
-					(reference "#PWR017")
+					(reference "#PWR03")
 					(unit 1)
 				)
@@
 		(dnp no)
 		(fields_autoplaced yes)
-		(property "Reference" "#PWR016"
+		(property "Reference" "#PWR01"
 			(at 204.47 20.32 0)
 			(hide yes)
@@
 			(project "PMM-1.0-R1"
 				(path "/dfbd1ee6-4059-4519-bc2e-4814be9dda35"
-					(reference "#PWR016")
+					(reference "#PWR01")
 					(unit 1)
 				)
@@
 		(dnp no)
 		(fields_autoplaced yes)
-		(property "Reference" "U3"
+		(property "Reference" "U1"
 			(at 235.8233 19.05 0)
 			(show_name no)
@@
 			(project "PMM-1.0-R1"
 				(path "/dfbd1ee6-4059-4519-bc2e-4814be9dda35"
-					(reference "U3")
+					(reference "U1")
 					(unit 1)
 				)
@@
 		(dnp no)
 		(fields_autoplaced yes)
-		(property "Reference" "#PWR039"
+		(property "Reference" "#PWR02"
 			(at 204.47 31.75 0)
 			(hide yes)
@@
 			(project "PMM-1.0-R1"
 				(path "/dfbd1ee6-4059-4519-bc2e-4814be9dda35"
-					(reference "#PWR039")
+					(reference "#PWR02")
 					(unit 1)
 				)
@@
 	)
 	(sheet
-		(at 67.31 45.72)
+		(at 76.2 25.4)
 		(size 12.7 5.08)
 		(exclude_from_sim no)
@@
 		)
 		(property "Sheetname" "TPS61089"
-			(at 67.31 45.0084 0)
+			(at 76.2 24.6884 0)
 			(show_name no)
 			(do_not_autoplace no)
@@
 		)
 		(property "Sheetfile" "tps61089.kicad_sch"
-			(at 67.31 51.3846 0)
+			(at 76.2 31.0646 0)
 			(show_name no)
 			(do_not_autoplace no)
@@
 		)
 		(pin "VIN" input
-			(at 67.31 48.26 180)
+			(at 76.2 27.94 180)
 			(effects
 				(font
@@
 		)
 		(pin "VOUT" input
-			(at 80.01 48.26 0)
+			(at 88.9 27.94 0)
 			(effects
 				(font
@@
 	)
 	(sheet
-		(at 165.1 50.8)
+		(at 101.6 25.4)
 		(size 12.7 12.7)
 		(exclude_from_sim no)
@@
 		)
 		(property "Sheetname" "TLV75733"
-			(at 165.1 50.0884 0)
+			(at 101.6 24.6884 0)
 			(show_name no)
 			(do_not_autoplace no)
@@
 		)
 		(property "Sheetfile" "tlv75733.kicad_sch"
-			(at 165.1 64.0846 0)
+			(at 101.6 38.6846 0)
 			(show_name no)
 			(do_not_autoplace no)
@@
 		)
 		(pin "VIN" input
-			(at 165.1 53.34 180)
+			(at 101.6 27.94 180)
 			(effects
 				(font
@@
 		)
 		(pin "VOUT" input
-			(at 177.8 53.34 0)
+			(at 114.3 27.94 0)
 			(effects
 				(font
@@
 	)
 	(sheet
-		(at 43.18 25.4)
+		(at 50.8 63.5)
 		(size 12.7 12.7)
 		(exclude_from_sim no)
@@
 		)
 		(property "Sheetname" "BQ25895"
-			(at 43.18 24.6884 0)
+			(at 50.8 62.7884 0)
 			(show_name no)
 			(do_not_autoplace no)
@@
 		)
 		(property "Sheetfile" "bq25895.kicad_sch"
-			(at 43.18 38.6846 0)
+			(at 50.8 76.7846 0)
 			(show_name no)
 			(do_not_autoplace no)
@@
 		)
 		(pin "BAT+" input
-			(at 43.18 27.94 180)
+			(at 50.8 66.04 180)
 			(effects
 				(font
@@
 		)
 		(pin "CE" input
-			(at 55.88 27.94 0)
+			(at 63.5 66.04 0)
 			(effects
 				(font
@@
 		)
 		(pin "INT" input
-			(at 55.88 30.48 0)
+			(at 63.5 68.58 0)
 			(effects
 				(font
@@
 		)
 		(pin "OTG" input
-			(at 43.18 35.56 180)
+			(at 50.8 73.66 180)
 			(effects
 				(font
@@
 		)
 		(pin "SCL" input
-			(at 55.88 33.02 0)
+			(at 63.5 71.12 0)
 			(effects
 				(font
@@
 		)
 		(pin "SDA" input
-			(at 55.88 35.56 0)
+			(at 63.5 73.66 0)
 			(effects
 				(font
@@
 		)
 		(pin "VIN" input
-			(at 43.18 30.48 180)
+			(at 50.8 68.58 180)
 			(effects
 				(font
@@
 		)
 		(pin "VOUT" input
-			(at 43.18 33.02 180)
+			(at 50.8 71.12 180)
 			(effects
 				(font
@@
 	)
 	(sheet
-		(at 92.71 45.72)
+		(at 101.6 50.8)
 		(size 12.7 11.43)
 		(exclude_from_sim no)
@@
 		)
 		(property "Sheetname" "TPS22917"
-			(at 92.71 45.0084 0)
+			(at 101.6 50.0884 0)
 			(show_name no)
 			(do_not_autoplace no)
@@
 		)
 		(property "Sheetfile" "tps22917.kicad_sch"
-			(at 92.71 57.7346 0)
+			(at 101.6 62.8146 0)
 			(show_name no)
 			(do_not_autoplace no)
@@
 		)
 		(pin "ON" input
-			(at 92.71 54.61 180)
+			(at 101.6 59.69 180)
 			(effects
 				(font
@@
 		)
 		(pin "VIN" input
-			(at 92.71 48.26 180)
+			(at 101.6 53.34 180)
 			(effects
 				(font
@@
 		)
 		(pin "VOUT" input
-			(at 105.41 48.26 0)
+			(at 114.3 53.34 0)
 			(effects
 				(font
@@
 	)
 	(sheet
-		(at 36.83 45.72)
+		(at 38.1 25.4)
 		(size 25.4 10.16)
 		(exclude_from_sim no)
@@
 		)
 		(property "Sheetname" "BQ27441"
-			(at 36.83 45.0084 0)
+			(at 38.1 24.6884 0)
 			(show_name no)
 			(do_not_autoplace no)
@@
 		)
 		(property "Sheetfile" "bq27441.kicad_sch"
-			(at 36.83 56.4646 0)
+			(at 38.1 36.1446 0)
 			(show_name no)
 			(do_not_autoplace no)
@@
 		)
 		(pin "BATTOUT" input
-			(at 62.23 48.26 0)
+			(at 63.5 27.94 0)
 			(effects
 				(font
@@
 		)
 		(pin "GPOUT" input
-			(at 36.83 48.26 180)
+			(at 38.1 27.94 180)
 			(effects
 				(font
@@
 		)
 		(pin "PACK+" input
-			(at 36.83 50.8 180)
+			(at 38.1 30.48 180)
 			(effects
 				(font
@@
 		)
 		(pin "PACK-" input
-			(at 36.83 53.34 180)
+			(at 38.1 33.02 180)
 			(effects
 				(font
@@
 		)
 		(pin "SCL" input
-			(at 62.23 50.8 0)
+			(at 63.5 30.48 0)
 			(effects
 				(font
@@
 		)
 		(pin "SDA" input
-			(at 62.23 53.34 0)
-			(effects
-				(font
+			(at 63.5 33.02 0)
+			(effects
+				(font

Commit message: finished schematics
Parts:
- removed C1: 100nF, symbol Device:C_Small
- removed U1: STM32C031C4T6, Package_QFP:LQFP-48_7x7mm_P0.5mm, symbol MCU_ST_STM32C0:STM32C031C4Tx
- added A1: PMM, PMM:PMM, symbol PMM:PMM
- added D1: LED, symbol Device:LED
- added R1: 10k, symbol Device:R_Small_US
Connections:
- net +3.3V: now also A1.11 (3V3), D1.2 (A)
- net GND: now also A1.1 (GND), A1.10 (GND), A1.12 (GND), A1.2 (GND), A1.21 (GND), A1.22 (GND), R1.2
- new net: D1.1 (K), R1.1
- new net 5V_OUT: A1.7 (5V_OUT), A1.8 (5V_OUT), A1.9 (5V_OUT)
- new net ADC_IN: A1.31 (ADC_IN)
- new net BATT+: A1.3 (VBAT+), A1.4 (VBAT+)
- new net FORCE_ON: A1.18 (FORCE_ON)
- new net PMM_INT: A1.15 (PMM_INIT)
- new net SCL: A1.14 (SCL)
- new net SDA: A1.13 (SDA)
- new net SHDN: A1.17 (SHDN)
- new net SWCLK: A1.39 (SWCLK)
- new net SWDIO: A1.40 (SWDIO)
- new net UART_RX: A1.36 (UART_RX)
- new net UART_TX: A1.37 (UART_TX)
- new net VBUS_5V_IN: A1.5 (VBAT_5V_IN), A1.6 (VBAT_5V_IN)
- no-connect marks 0 -> 16
Other:
- added sheet STM32 (stm32.kicad_sch)
