File: kicad/bq25895.kicad_sch (KiCad schematic)
At the start: 19 parts, among them U1 BQ25895RTW

Commit message: update gitignore and whatnot
Parts:
- renumbered C1 to C19, C2 to C20, C3 to C21, C4 to C22, C5 to C23, C6 to C24, L1 to L2, R1 to R10, R2 to R11, R3 to R12, R4 to R13, R5 to R14, R6 to R15, R7 to R16, R8 to R17, R9 to R18, U1 to U5

Commit message: finished schematics
Parts:
- added TP1, TP2: TestPoint, symbol Connector:TestPoint
- renumbered C19 to C18, C20 to C19, C21 to C20, C22 to C21, C23 to C22, C24 to C23, D1 to D2, R10 to R11, R11 to R12, R12 to R13, R13 to R14, R14 to R15, R15 to R16, R16 to R17, R17 to R18, R18 to R19, U5 to U4
Connections:
- net at U4.2 (D+): now also TP2.1; no longer U4.3 (D-)
- new net: TP1.1, U4.3 (D-)
