File: kicad/tlv75733.kicad_sch (KiCad schematic)
At the start: 4 parts, among them U2 TLV75733PDBV

Commit message: update gitignore and whatnot
Parts:
- renumbered C7 to C25, C8 to C26, C9 to C27, U2 to U6
Changed lines of the file:
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@@
 		(dnp no)
 		(fields_autoplaced yes)
-		(property "Reference" "#PWR015"
+		(property "Reference" "#PWR039"
 			(at 44.45 50.8 0)
 			(hide yes)
@@
 			(project "PMM-1.0-R1"
 				(path "/dfbd1ee6-4059-4519-bc2e-4814be9dda35/345fcbde-0403-4e9a-a959-8171526cc73f"
-					(reference "#PWR015")
+					(reference "#PWR039")
 					(unit 1)
 				)
@@
 		(dnp no)
 		(fields_autoplaced yes)
-		(property "Reference" "C8"
+		(property "Reference" "C26"
 			(at 63.5 34.2962 0)
 			(show_name no)
@@
 			(project "PMM-1.0-R1"
 				(path "/dfbd1ee6-4059-4519-bc2e-4814be9dda35/345fcbde-0403-4e9a-a959-8171526cc73f"
-					(reference "C8")
+					(reference "C26")
 					(unit 1)
 				)
@@
 		(dnp no)
 		(fields_autoplaced yes)
-		(property "Reference" "U2"
+		(property "Reference" "U6"
 			(at 44.45 25.4 0)
 			(show_name no)
@@
 			(project "PMM-1.0-R1"
 				(path "/dfbd1ee6-4059-4519-bc2e-4814be9dda35/345fcbde-0403-4e9a-a959-8171526cc73f"
-					(reference "U2")
+					(reference "U6")
 					(unit 1)
 				)
@@
 		(dnp no)
 		(fields_autoplaced yes)
-		(property "Reference" "C7"
+		(property "Reference" "C25"
 			(at 30.48 34.2962 0)
 			(show_name no)
@@
 			(project "PMM-1.0-R1"
 				(path "/dfbd1ee6-4059-4519-bc2e-4814be9dda35/345fcbde-0403-4e9a-a959-8171526cc73f"
-					(reference "C7")
+					(reference "C25")
 					(unit 1)
 				)
@@
 		(dnp no)
 		(fields_autoplaced yes)
-		(property "Reference" "C9"
+		(property "Reference" "C27"
 			(at 74.93 34.2962 0)
 			(show_name no)
@@
 			(project "PMM-1.0-R1"
 				(path "/dfbd1ee6-4059-4519-bc2e-4814be9dda35/345fcbde-0403-4e9a-a959-8171526cc73f"
-					(reference "C9")
-					(unit 1)
-				)
+					(reference "C27")
+					(unit 1)
+				)

Commit message: finished schematics
Parts:
- renumbered C25 to C24, C26 to C25, C27 to C26, U6 to U5
Changed lines of the file:
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@@
 		(dnp no)
 		(fields_autoplaced yes)
-		(property "Reference" "#PWR039"
+		(property "Reference" "#PWR045"
 			(at 44.45 50.8 0)
 			(hide yes)
@@
 			(project "PMM-1.0-R1"
 				(path "/dfbd1ee6-4059-4519-bc2e-4814be9dda35/345fcbde-0403-4e9a-a959-8171526cc73f"
-					(reference "#PWR039")
+					(reference "#PWR045")
 					(unit 1)
 				)
@@
 		(dnp no)
 		(fields_autoplaced yes)
-		(property "Reference" "C26"
+		(property "Reference" "C25"
 			(at 63.5 34.2962 0)
 			(show_name no)
@@
 			(project "PMM-1.0-R1"
 				(path "/dfbd1ee6-4059-4519-bc2e-4814be9dda35/345fcbde-0403-4e9a-a959-8171526cc73f"
-					(reference "C26")
+					(reference "C25")
 					(unit 1)
 				)
@@
 		(dnp no)
 		(fields_autoplaced yes)
-		(property "Reference" "U6"
+		(property "Reference" "U5"
 			(at 44.45 25.4 0)
 			(show_name no)
@@
 			(project "PMM-1.0-R1"
 				(path "/dfbd1ee6-4059-4519-bc2e-4814be9dda35/345fcbde-0403-4e9a-a959-8171526cc73f"
-					(reference "U6")
+					(reference "U5")
 					(unit 1)
 				)
@@
 		(dnp no)
 		(fields_autoplaced yes)
-		(property "Reference" "C25"
+		(property "Reference" "C24"
 			(at 30.48 34.2962 0)
 			(show_name no)
@@
 			(project "PMM-1.0-R1"
 				(path "/dfbd1ee6-4059-4519-bc2e-4814be9dda35/345fcbde-0403-4e9a-a959-8171526cc73f"
-					(reference "C25")
+					(reference "C24")
 					(unit 1)
 				)
@@
 		(dnp no)
 		(fields_autoplaced yes)
-		(property "Reference" "C27"
+		(property "Reference" "C26"
 			(at 74.93 34.2962 0)
 			(show_name no)
@@
 			(project "PMM-1.0-R1"
 				(path "/dfbd1ee6-4059-4519-bc2e-4814be9dda35/345fcbde-0403-4e9a-a959-8171526cc73f"
-					(reference "C27")
-					(unit 1)
-				)
+					(reference "C26")
+					(unit 1)
+				)
