File: kicad/tps22917.kicad_sch (KiCad schematic)
At the start: 7 parts, among them U5 TPS22917DBV

Commit message: update gitignore and whatnot
Parts:
- renumbered C21 to C13, C22 to C14, C23 to C15, C24 to C16, R15 to R6, R16 to R7, U5 to U3
Changed lines of the file:
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@@
 		(dnp no)
 		(fields_autoplaced yes)
-		(property "Reference" "#PWR030"
+		(property "Reference" "#PWR016"
 			(at 25.4 54.61 0)
 			(hide yes)
@@
 			(project "PMM-1.0-R1"
 				(path "/dfbd1ee6-4059-4519-bc2e-4814be9dda35/b58734b6-a6f6-4547-b140-16953b8cb461"
-					(reference "#PWR030")
+					(reference "#PWR016")
 					(unit 1)
 				)
@@
 		(dnp no)
 		(fields_autoplaced yes)
-		(property "Reference" "C22"
+		(property "Reference" "C14"
 			(at 39.37 43.1862 0)
 			(show_name no)
@@
 			(project "PMM-1.0-R1"
 				(path "/dfbd1ee6-4059-4519-bc2e-4814be9dda35/b58734b6-a6f6-4547-b140-16953b8cb461"
-					(reference "C22")
+					(reference "C14")
 					(unit 1)
 				)
@@
 		(dnp no)
 		(fields_autoplaced yes)
-		(property "Reference" "C21"
+		(property "Reference" "C13"
 			(at 27.94 43.1862 0)
 			(show_name no)
@@
 			(project "PMM-1.0-R1"
 				(path "/dfbd1ee6-4059-4519-bc2e-4814be9dda35/b58734b6-a6f6-4547-b140-16953b8cb461"
-					(reference "C21")
+					(reference "C13")
 					(unit 1)
 				)
@@
 		(dnp no)
 		(fields_autoplaced yes)
-		(property "Reference" "#PWR034"
+		(property "Reference" "#PWR020"
 			(at 91.44 54.61 0)
 			(hide yes)
@@
 			(project "PMM-1.0-R1"
 				(path "/dfbd1ee6-4059-4519-bc2e-4814be9dda35/b58734b6-a6f6-4547-b140-16953b8cb461"
-					(reference "#PWR034")
+					(reference "#PWR020")
 					(unit 1)
 				)
@@
 		(dnp no)
 		(fields_autoplaced yes)
-		(property "Reference" "C23"
+		(property "Reference" "C15"
 			(at 49.53 41.9162 0)
 			(show_name no)
@@
 			(project "PMM-1.0-R1"
 				(path "/dfbd1ee6-4059-4519-bc2e-4814be9dda35/b58734b6-a6f6-4547-b140-16953b8cb461"
-					(reference "C23")
+					(reference "C15")
 					(unit 1)
 				)
@@
 		(dnp no)
 		(fields_autoplaced yes)
-		(property "Reference" "#PWR031"
+		(property "Reference" "#PWR017"
 			(at 36.83 54.61 0)
 			(hide yes)
@@
 			(project "PMM-1.0-R1"
 				(path "/dfbd1ee6-4059-4519-bc2e-4814be9dda35/b58734b6-a6f6-4547-b140-16953b8cb461"
-					(reference "#PWR031")
+					(reference "#PWR017")
 					(unit 1)
 				)
@@
 		(dnp no)
 		(fields_autoplaced yes)
-		(property "Reference" "#PWR033"
+		(property "Reference" "#PWR019"
 			(at 66.04 58.42 0)
 			(hide yes)
@@
 			(project "PMM-1.0-R1"
 				(path "/dfbd1ee6-4059-4519-bc2e-4814be9dda35/b58734b6-a6f6-4547-b140-16953b8cb461"
-					(reference "#PWR033")
+					(reference "#PWR019")
 					(unit 1)
 				)
@@
 		(dnp no)
 		(fields_autoplaced yes)
-		(property "Reference" "R16"
+		(property "Reference" "R7"
 			(at 83.82 43.1799 0)
 			(show_name no)
@@
 			(project "PMM-1.0-R1"
 				(path "/dfbd1ee6-4059-4519-bc2e-4814be9dda35/b58734b6-a6f6-4547-b140-16953b8cb461"
-					(reference "R16")
+					(reference "R7")
 					(unit 1)
 				)
@@
 		(dnp no)
 		(fields_autoplaced yes)
-		(property "Reference" "R15"
+		(property "Reference" "R6"
 			(at 58.42 52.0699 0)
 			(show_name no)
@@
 			(project "PMM-1.0-R1"
 				(path "/dfbd1ee6-4059-4519-bc2e-4814be9dda35/b58734b6-a6f6-4547-b140-16953b8cb461"
-					(reference "R15")
+					(reference "R6")
 					(unit 1)
 				)
@@
 		(dnp no)
 		(fields_autoplaced yes)
-		(property "Reference" "U5"
+		(property "Reference" "U3"
 			(at 66.04 33.02 0)
 			(show_name no)
@@
 			(project "PMM-1.0-R1"
 				(path "/dfbd1ee6-4059-4519-bc2e-4814be9dda35/b58734b6-a6f6-4547-b140-16953b8cb461"
-					(reference "U5")
+					(reference "U3")
 					(unit 1)
 				)
@@
 		(dnp no)
 		(fields_autoplaced yes)
-		(property "Reference" "C24"
+		(property "Reference" "C16"
 			(at 93.98 43.1862 0)
 			(show_name no)
@@
 			(project "PMM-1.0-R1"
 				(path "/dfbd1ee6-4059-4519-bc2e-4814be9dda35/b58734b6-a6f6-4547-b140-16953b8cb461"
-					(reference "C24")
+					(reference "C16")
 					(unit 1)
 				)
@@
 		(dnp no)
 		(fields_autoplaced yes)
-		(property "Reference" "#PWR032"
+		(property "Reference" "#PWR018"
 			(at 55.88 63.5 0)
 			(hide yes)
@@
 			(project "PMM-1.0-R1"
 				(path "/dfbd1ee6-4059-4519-bc2e-4814be9dda35/b58734b6-a6f6-4547-b140-16953b8cb461"
-					(reference "#PWR032")
-					(unit 1)
-				)
+					(reference "#PWR018")
+					(unit 1)
+				)

Commit message: finished schematics
Parts:
- renumbered C13 to C12, C14 to C13, C15 to C14, C16 to C15, R6 to R7, R7 to R8, U3 to U2
Changed lines of the file:
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@@
 		(dnp no)
 		(fields_autoplaced yes)
-		(property "Reference" "#PWR016"
+		(property "Reference" "#PWR022"
 			(at 25.4 54.61 0)
 			(hide yes)
@@
 			(project "PMM-1.0-R1"
 				(path "/dfbd1ee6-4059-4519-bc2e-4814be9dda35/b58734b6-a6f6-4547-b140-16953b8cb461"
-					(reference "#PWR016")
+					(reference "#PWR022")
 					(unit 1)
 				)
@@
 		(dnp no)
 		(fields_autoplaced yes)
-		(property "Reference" "C14"
+		(property "Reference" "C13"
 			(at 39.37 43.1862 0)
 			(show_name no)
@@
 			(project "PMM-1.0-R1"
 				(path "/dfbd1ee6-4059-4519-bc2e-4814be9dda35/b58734b6-a6f6-4547-b140-16953b8cb461"
-					(reference "C14")
+					(reference "C13")
 					(unit 1)
 				)
@@
 		(dnp no)
 		(fields_autoplaced yes)
-		(property "Reference" "C13"
+		(property "Reference" "C12"
 			(at 27.94 43.1862 0)
 			(show_name no)
@@
 			(project "PMM-1.0-R1"
 				(path "/dfbd1ee6-4059-4519-bc2e-4814be9dda35/b58734b6-a6f6-4547-b140-16953b8cb461"
-					(reference "C13")
+					(reference "C12")
 					(unit 1)
 				)
@@
 		(dnp no)
 		(fields_autoplaced yes)
-		(property "Reference" "#PWR020"
+		(property "Reference" "#PWR026"
 			(at 91.44 54.61 0)
 			(hide yes)
@@
 			(project "PMM-1.0-R1"
 				(path "/dfbd1ee6-4059-4519-bc2e-4814be9dda35/b58734b6-a6f6-4547-b140-16953b8cb461"
-					(reference "#PWR020")
+					(reference "#PWR026")
 					(unit 1)
 				)
@@
 		(dnp no)
 		(fields_autoplaced yes)
-		(property "Reference" "C15"
+		(property "Reference" "C14"
 			(at 49.53 41.9162 0)
 			(show_name no)
@@
 			(project "PMM-1.0-R1"
 				(path "/dfbd1ee6-4059-4519-bc2e-4814be9dda35/b58734b6-a6f6-4547-b140-16953b8cb461"
-					(reference "C15")
+					(reference "C14")
 					(unit 1)
 				)
@@
 		(dnp no)
 		(fields_autoplaced yes)
-		(property "Reference" "#PWR017"
+		(property "Reference" "#PWR023"
 			(at 36.83 54.61 0)
 			(hide yes)
@@
 			(project "PMM-1.0-R1"
 				(path "/dfbd1ee6-4059-4519-bc2e-4814be9dda35/b58734b6-a6f6-4547-b140-16953b8cb461"
-					(reference "#PWR017")
+					(reference "#PWR023")
 					(unit 1)
 				)
@@
 		(dnp no)
 		(fields_autoplaced yes)
-		(property "Reference" "#PWR019"
+		(property "Reference" "#PWR025"
 			(at 66.04 58.42 0)
 			(hide yes)
@@
 			(project "PMM-1.0-R1"
 				(path "/dfbd1ee6-4059-4519-bc2e-4814be9dda35/b58734b6-a6f6-4547-b140-16953b8cb461"
-					(reference "#PWR019")
+					(reference "#PWR025")
 					(unit 1)
 				)
@@
 		(dnp no)
 		(fields_autoplaced yes)
-		(property "Reference" "R7"
+		(property "Reference" "R8"
 			(at 83.82 43.1799 0)
 			(show_name no)
@@
 			(project "PMM-1.0-R1"
 				(path "/dfbd1ee6-4059-4519-bc2e-4814be9dda35/b58734b6-a6f6-4547-b140-16953b8cb461"
-					(reference "R7")
+					(reference "R8")
 					(unit 1)
 				)
@@
 		(dnp no)
 		(fields_autoplaced yes)
-		(property "Reference" "R6"
+		(property "Reference" "R7"
 			(at 58.42 52.0699 0)
 			(show_name no)
@@
 			(project "PMM-1.0-R1"
 				(path "/dfbd1ee6-4059-4519-bc2e-4814be9dda35/b58734b6-a6f6-4547-b140-16953b8cb461"
-					(reference "R6")
+					(reference "R7")
 					(unit 1)
 				)
@@
 		(dnp no)
 		(fields_autoplaced yes)
-		(property "Reference" "U3"
+		(property "Reference" "U2"
 			(at 66.04 33.02 0)
 			(show_name no)
@@
 			(project "PMM-1.0-R1"
 				(path "/dfbd1ee6-4059-4519-bc2e-4814be9dda35/b58734b6-a6f6-4547-b140-16953b8cb461"
-					(reference "U3")
+					(reference "U2")
 					(unit 1)
 				)
@@
 		(dnp no)
 		(fields_autoplaced yes)
-		(property "Reference" "C16"
+		(property "Reference" "C15"
 			(at 93.98 43.1862 0)
 			(show_name no)
@@
 			(project "PMM-1.0-R1"
 				(path "/dfbd1ee6-4059-4519-bc2e-4814be9dda35/b58734b6-a6f6-4547-b140-16953b8cb461"
-					(reference "C16")
+					(reference "C15")
 					(unit 1)
 				)
@@
 		(dnp no)
 		(fields_autoplaced yes)
-		(property "Reference" "#PWR018"
+		(property "Reference" "#PWR024"
 			(at 55.88 63.5 0)
 			(hide yes)
@@
 			(project "PMM-1.0-R1"
 				(path "/dfbd1ee6-4059-4519-bc2e-4814be9dda35/b58734b6-a6f6-4547-b140-16953b8cb461"
-					(reference "#PWR018")
-					(unit 1)
-				)
+					(reference "#PWR024")
+					(unit 1)
+				)
