File: kicad/tps61089.kicad_sch (KiCad schematic)
At the start: 18 parts, among them U4 TPS61089

Commit message: update gitignore and whatnot
Parts:
- renumbered C18 to C10, C19 to C11, C20 to C12, C10 to C2, C11 to C3, C12 to C4, C13 to C5, C14 to C6, C15 to C7, C16 to C8, C17 to C9, L2 to L1, R10 to R1, R11 to R2, R12 to R3, R13 to R4, R14 to R5, U4 to U2

Commit message: finished schematics
Parts:
- renumbered C2 to C1, C11 to C10, C12 to C11, C3 to C2, C4 to C3, C5 to C4, C6 to C5, C7 to C6, C8 to C7, C9 to C8, C10 to C9, R1 to R2, R2 to R3, R3 to R4, R4 to R5, R5 to R6, U2 to U1
Changed lines of the file:
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@@
 		(dnp no)
 		(fields_autoplaced yes)
-		(property "Reference" "#PWR015"
+		(property "Reference" "#PWR021"
 			(at 158.75 64.77 0)
 			(hide yes)
@@
 			(project "PMM-1.0-R1"
 				(path "/dfbd1ee6-4059-4519-bc2e-4814be9dda35/1bb64621-37a6-4f79-84fe-8a9a999dcffc"
-					(reference "#PWR015")
+					(reference "#PWR021")
 					(unit 1)
 				)
@@
 		(dnp no)
 		(fields_autoplaced yes)
-		(property "Reference" "#PWR014"
+		(property "Reference" "#PWR020"
 			(at 139.7 77.47 0)
 			(hide yes)
@@
 			(project "PMM-1.0-R1"
 				(path "/dfbd1ee6-4059-4519-bc2e-4814be9dda35/1bb64621-37a6-4f79-84fe-8a9a999dcffc"
-					(reference "#PWR014")
+					(reference "#PWR020")
 					(unit 1)
 				)
@@
 		(dnp no)
 		(fields_autoplaced yes)
-		(property "Reference" "#PWR013"
+		(property "Reference" "#PWR019"
 			(at 137.16 50.8 0)
 			(hide yes)
@@
 			(project "PMM-1.0-R1"
 				(path "/dfbd1ee6-4059-4519-bc2e-4814be9dda35/1bb64621-37a6-4f79-84fe-8a9a999dcffc"
-					(reference "#PWR013")
+					(reference "#PWR019")
 					(unit 1)
 				)
@@
 		(dnp no)
 		(fields_autoplaced yes)
-		(property "Reference" "C8"
+		(property "Reference" "C7"
 			(at 118.11 39.3762 0)
 			(show_name no)
@@
 			(project "PMM-1.0-R1"
 				(path "/dfbd1ee6-4059-4519-bc2e-4814be9dda35/1bb64621-37a6-4f79-84fe-8a9a999dcffc"
-					(reference "C8")
+					(reference "C7")
 					(unit 1)
 				)
@@
 		(dnp no)
 		(fields_autoplaced yes)
-		(property "Reference" "C10"
+		(property "Reference" "C9"
 			(at 135.89 60.9662 0)
 			(show_name no)
@@
 			(project "PMM-1.0-R1"
 				(path "/dfbd1ee6-4059-4519-bc2e-4814be9dda35/1bb64621-37a6-4f79-84fe-8a9a999dcffc"
-					(reference "C10")
+					(reference "C9")
 					(unit 1)
 				)
@@
 		(dnp no)
 		(fields_autoplaced yes)
-		(property "Reference" "C9"
+		(property "Reference" "C8"
 			(at 129.54 39.3762 0)
 			(show_name no)
@@
 			(project "PMM-1.0-R1"
 				(path "/dfbd1ee6-4059-4519-bc2e-4814be9dda35/1bb64621-37a6-4f79-84fe-8a9a999dcffc"
-					(reference "C9")
+					(reference "C8")
 					(unit 1)
 				)
@@
 		(dnp no)
 		(fields_autoplaced yes)
-		(property "Reference" "#PWR09"
+		(property "Reference" "#PWR015"
 			(at 113.03 74.93 0)
 			(hide yes)
@@
 			(project "PMM-1.0-R1"
 				(path "/dfbd1ee6-4059-4519-bc2e-4814be9dda35/1bb64621-37a6-4f79-84fe-8a9a999dcffc"
-					(reference "#PWR09")
+					(reference "#PWR015")
 					(unit 1)
 				)
@@
 		(dnp no)
 		(fields_autoplaced yes)
-		(property "Reference" "C7"
+		(property "Reference" "C6"
 			(at 115.57 63.5062 0)
 			(show_name no)
@@
 			(project "PMM-1.0-R1"
 				(path "/dfbd1ee6-4059-4519-bc2e-4814be9dda35/1bb64621-37a6-4f79-84fe-8a9a999dcffc"
-					(reference "C7")
+					(reference "C6")
 					(unit 1)
 				)
@@
 		(dnp no)
 		(fields_autoplaced yes)
-		(property "Reference" "C3"
+		(property "Reference" "C2"
 			(at 39.37 48.2662 0)
 			(show_name no)
@@
 			(project "PMM-1.0-R1"
 				(path "/dfbd1ee6-4059-4519-bc2e-4814be9dda35/1bb64621-37a6-4f79-84fe-8a9a999dcffc"
-					(reference "C3")
+					(reference "C2")
 					(unit 1)
 				)
@@
 		(dnp no)
 		(fields_autoplaced yes)
-		(property "Reference" "#PWR05"
+		(property "Reference" "#PWR011"
 			(at 36.83 59.69 0)
 			(hide yes)
@@
 			(project "PMM-1.0-R1"
 				(path "/dfbd1ee6-4059-4519-bc2e-4814be9dda35/1bb64621-37a6-4f79-84fe-8a9a999dcffc"
-					(reference "#PWR05")
+					(reference "#PWR011")
 					(unit 1)
 				)
@@
 		(dnp no)
 		(fields_autoplaced yes)
-		(property "Reference" "#PWR012"
+		(property "Reference" "#PWR018"
 			(at 127 50.8 0)
 			(hide yes)
@@
 			(project "PMM-1.0-R1"
 				(path "/dfbd1ee6-4059-4519-bc2e-4814be9dda35/1bb64621-37a6-4f79-84fe-8a9a999dcffc"
-					(reference "#PWR012")
+					(reference "#PWR018")
 					(unit 1)
 				)
@@
 		(dnp no)
 		(fields_autoplaced yes)
-		(property "Reference" "R3"
+		(property "Reference" "R4"
 			(at 144.78 58.4199 0)
 			(show_name no)
@@
 			(project "PMM-1.0-R1"
 				(path "/dfbd1ee6-4059-4519-bc2e-4814be9dda35/1bb64621-37a6-4f79-84fe-8a9a999dcffc"
-					(reference "R3")
+					(reference "R4")
 					(unit 1)
 				)
@@
 		(dnp no)
 		(fields_autoplaced yes)
-		(property "Reference" "#PWR04"
+		(property "Reference" "#PWR010"
 			(at 26.67 59.69 0)
 			(hide yes)
@@
 			(project "PMM-1.0-R1"
 				(path "/dfbd1ee6-4059-4519-bc2e-4814be9dda35/1bb64621-37a6-4f79-84fe-8a9a999dcffc"
-					(reference "#PWR04")
+					(reference "#PWR010")
 					(unit 1)
 				)
@@
 		(dnp no)
 		(fields_autoplaced yes)
-		(property "Reference" "R1"
+		(property "Reference" "R2"
 			(at 76.2 48.2599 0)
 			(show_name no)
@@
 			(project "PMM-1.0-R1"
 				(path "/dfbd1ee6-4059-4519-bc2e-4814be9dda35/1bb64621-37a6-4f79-84fe-8a9a999dcffc"
-					(reference "R1")
+					(reference "R2")
 					(unit 1)
 				)
@@
 		(dnp no)
 		(fields_autoplaced yes)
-		(property "Reference" "R5"
+		(property "Reference" "R6"
 			(at 161.29 53.3399 0)
 			(show_name no)
@@
 			(project "PMM-1.0-R1"
 				(path "/dfbd1ee6-4059-4519-bc2e-4814be9dda35/1bb64621-37a6-4f79-84fe-8a9a999dcffc"
-					(reference "R5")
+					(reference "R6")
 					(unit 1)
 				)
@@
 		(dnp no)
 		(fields_autoplaced yes)
-		(property "Reference" "R2"
+		(property "Reference" "R3"
 			(at 127 63.4999 0)
 			(show_name no)
@@
 			(project "PMM-1.0-R1"
 				(path "/dfbd1ee6-4059-4519-bc2e-4814be9dda35/1bb64621-37a6-4f79-84fe-8a9a999dcffc"
-					(reference "R2")
+					(reference "R3")
 					(unit 1)
 				)
@@
 		(dnp no)
 		(fields_autoplaced yes)
-		(property "Reference" "C6"
+		(property "Reference" "C5"
 			(at 86.36 48.2662 0)
 			(show_name no)
@@
 			(project "PMM-1.0-R1"
 				(path "/dfbd1ee6-4059-4519-bc2e-4814be9dda35/1bb64621-37a6-4f79-84fe-8a9a999dcffc"
-					(reference "C6")
+					(reference "C5")
 					(unit 1)
 				)
@@
 		(dnp no)
 		(fields_autoplaced yes)
-		(property "Reference" "R4"
+		(property "Reference" "R5"
 			(at 161.29 45.7199 0)
 			(show_name no)
@@
 			(project "PMM-1.0-R1"
 				(path "/dfbd1ee6-4059-4519-bc2e-4814be9dda35/1bb64621-37a6-4f79-84fe-8a9a999dcffc"
-					(reference "R4")
+					(reference "R5")
 					(unit 1)
 				)
@@
 		(dnp no)
 		(fields_autoplaced yes)
-		(property "Reference" "#PWR011"
+		(property "Reference" "#PWR017"
 			(at 124.46 74.93 0)
 			(hide yes)
@@
 			(project "PMM-1.0-R1"
 				(path "/dfbd1ee6-4059-4519-bc2e-4814be9dda35/1bb64621-37a6-4f79-84fe-8a9a999dcffc"
-					(reference "#PWR011")
+					(reference "#PWR017")
 					(unit 1)
 				)
@@
 		(dnp no)
 		(fields_autoplaced yes)
-		(property "Reference" "#PWR07"
+		(property "Reference" "#PWR013"
 			(at 57.15 59.69 0)
 			(hide yes)
@@
 			(project "PMM-1.0-R1"
 				(path "/dfbd1ee6-4059-4519-bc2e-4814be9dda35/1bb64621-37a6-4f79-84fe-8a9a999dcffc"
-					(reference "#PWR07")
+					(reference "#PWR013")
 					(unit 1)
 				)
@@
 		(dnp no)
 		(fields_autoplaced yes)
-		(property "Reference" "C12"
+		(property "Reference" "C11"
 			(at 144.78 64.7762 0)
 			(show_name no)
@@
 			(project "PMM-1.0-R1"
 				(path "/dfbd1ee6-4059-4519-bc2e-4814be9dda35/1bb64621-37a6-4f79-84fe-8a9a999dcffc"
-					(reference "C12")
+					(reference "C11")
 					(unit 1)
 				)
@@
 		(dnp no)
 		(fields_autoplaced yes)
-		(property "Reference" "C5"
+		(property "Reference" "C4"
 			(at 59.69 48.2662 0)
 			(show_name no)
@@
 			(project "PMM-1.0-R1"
 				(path "/dfbd1ee6-4059-4519-bc2e-4814be9dda35/1bb64621-37a6-4f79-84fe-8a9a999dcffc"
-					(reference "C5")
+					(reference "C4")
 					(unit 1)
 				)
@@
 		(dnp no)
 		(fields_autoplaced yes)
-		(property "Reference" "C11"
+		(property "Reference" "C10"
 			(at 139.7 39.3762 0)
 			(show_name no)
@@
 			(project "PMM-1.0-R1"
 				(path "/dfbd1ee6-4059-4519-bc2e-4814be9dda35/1bb64621-37a6-4f79-84fe-8a9a999dcffc"
-					(reference "C11")
+					(reference "C10")
 					(unit 1)
 				)
@@
 		(dnp no)
 		(fields_autoplaced yes)
-		(property "Reference" "C2"
+		(property "Reference" "C1"
 			(at 29.21 48.2662 0)
 			(show_name no)
@@
 			(project "PMM-1.0-R1"
 				(path "/dfbd1ee6-4059-4519-bc2e-4814be9dda35/1bb64621-37a6-4f79-84fe-8a9a999dcffc"
-					(reference "C2")
+					(reference "C1")
 					(unit 1)
 				)
@@
 		(dnp no)
 		(fields_autoplaced yes)
-		(property "Reference" "C4"
+		(property "Reference" "C3"
 			(at 49.53 48.2662 0)
 			(show_name no)
@@
 			(project "PMM-1.0-R1"
 				(path "/dfbd1ee6-4059-4519-bc2e-4814be9dda35/1bb64621-37a6-4f79-84fe-8a9a999dcffc"
-					(reference "C4")
+					(reference "C3")
 					(unit 1)
 				)
@@
 		(dnp no)
 		(fields_autoplaced yes)
-		(property "Reference" "#PWR08"
+		(property "Reference" "#PWR014"
 			(at 100.33 73.66 0)
 			(hide yes)
@@
 			(project "PMM-1.0-R1"
 				(path "/dfbd1ee6-4059-4519-bc2e-4814be9dda35/1bb64621-37a6-4f79-84fe-8a9a999dcffc"
-					(reference "#PWR08")
+					(reference "#PWR014")
 					(unit 1)
 				)
@@
 		(dnp no)
 		(fields_autoplaced yes)
-		(property "Reference" "U2"
+		(property "Reference" "U1"
 			(at 100.33 38.1 0)
 			(show_name no)
@@
 			(project "PMM-1.0-R1"
 				(path "/dfbd1ee6-4059-4519-bc2e-4814be9dda35/1bb64621-37a6-4f79-84fe-8a9a999dcffc"
-					(reference "U2")
+					(reference "U1")
 					(unit 1)
 				)
@@
 		(dnp no)
 		(fields_autoplaced yes)
-		(property "Reference" "#PWR010"
+		(property "Reference" "#PWR016"
 			(at 115.57 50.8 0)
 			(hide yes)
@@
 			(project "PMM-1.0-R1"
 				(path "/dfbd1ee6-4059-4519-bc2e-4814be9dda35/1bb64621-37a6-4f79-84fe-8a9a999dcffc"
-					(reference "#PWR010")
+					(reference "#PWR016")
 					(unit 1)
 				)
@@
 		(dnp no)
 		(fields_autoplaced yes)
-		(property "Reference" "#PWR06"
+		(property "Reference" "#PWR012"
 			(at 46.99 59.69 0)
 			(hide yes)
@@
 			(project "PMM-1.0-R1"
 				(path "/dfbd1ee6-4059-4519-bc2e-4814be9dda35/1bb64621-37a6-4f79-84fe-8a9a999dcffc"
-					(reference "#PWR06")
-					(unit 1)
-				)
+					(reference "#PWR012")
+					(unit 1)
+				)
