File: kicad/bq27441.kicad_sch (KiCad schematic)
At the start: 5 parts, among them U6 BQ27441-G1

Commit message: update gitignore and whatnot
Parts:
- renumbered C25 to C17, C26 to C18, R17 to R8, R18 to R9, U6 to U4
Changed lines of the file:
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@@
 		(dnp no)
 		(fields_autoplaced yes)
-		(property "Reference" "#PWR035"
+		(property "Reference" "#PWR021"
 			(at 43.18 72.39 0)
 			(hide yes)
@@
 			(project "PMM-1.0-R1"
 				(path "/dfbd1ee6-4059-4519-bc2e-4814be9dda35/f17bf38e-84eb-4b8c-8211-b5a252381cf0"
-					(reference "#PWR035")
+					(reference "#PWR021")
 					(unit 1)
 				)
@@
 		(dnp no)
 		(fields_autoplaced yes)
-		(property "Reference" "#PWR036"
+		(property "Reference" "#PWR022"
 			(at 53.34 69.85 0)
 			(hide yes)
@@
 			(project "PMM-1.0-R1"
 				(path "/dfbd1ee6-4059-4519-bc2e-4814be9dda35/f17bf38e-84eb-4b8c-8211-b5a252381cf0"
-					(reference "#PWR036")
+					(reference "#PWR022")
 					(unit 1)
 				)
@@
 		(dnp no)
 		(fields_autoplaced yes)
-		(property "Reference" "C25"
+		(property "Reference" "C17"
 			(at 45.72 59.6962 0)
 			(show_name no)
@@
 			(project "PMM-1.0-R1"
 				(path "/dfbd1ee6-4059-4519-bc2e-4814be9dda35/f17bf38e-84eb-4b8c-8211-b5a252381cf0"
-					(reference "C25")
+					(reference "C17")
 					(unit 1)
 				)
@@
 		(dnp no)
 		(fields_autoplaced yes)
-		(property "Reference" "R18"
+		(property "Reference" "R9"
 			(at 55.88 58.4199 0)
 			(show_name no)
@@
 			(project "PMM-1.0-R1"
 				(path "/dfbd1ee6-4059-4519-bc2e-4814be9dda35/f17bf38e-84eb-4b8c-8211-b5a252381cf0"
-					(reference "R18")
+					(reference "R9")
 					(unit 1)
 				)
@@
 		(dnp no)
 		(fields_autoplaced yes)
-		(property "Reference" "#PWR037"
+		(property "Reference" "#PWR023"
 			(at 71.12 69.85 0)
 			(hide yes)
@@
 			(project "PMM-1.0-R1"
 				(path "/dfbd1ee6-4059-4519-bc2e-4814be9dda35/f17bf38e-84eb-4b8c-8211-b5a252381cf0"
-					(reference "#PWR037")
+					(reference "#PWR023")
 					(unit 1)
 				)
@@
 		(dnp no)
 		(fields_autoplaced yes)
-		(property "Reference" "C26"
+		(property "Reference" "C18"
 			(at 96.52 31.7562 0)
 			(show_name no)
@@
 			(project "PMM-1.0-R1"
 				(path "/dfbd1ee6-4059-4519-bc2e-4814be9dda35/f17bf38e-84eb-4b8c-8211-b5a252381cf0"
-					(reference "C26")
+					(reference "C18")
 					(unit 1)
 				)
@@
 		(dnp no)
 		(fields_autoplaced yes)
-		(property "Reference" "#PWR038"
+		(property "Reference" "#PWR024"
 			(at 93.98 43.18 0)
 			(hide yes)
@@
 			(project "PMM-1.0-R1"
 				(path "/dfbd1ee6-4059-4519-bc2e-4814be9dda35/f17bf38e-84eb-4b8c-8211-b5a252381cf0"
-					(reference "#PWR038")
+					(reference "#PWR024")
 					(unit 1)
 				)
@@
 		(dnp no)
 		(fields_autoplaced yes)
-		(property "Reference" "U6"
+		(property "Reference" "U4"
 			(at 72.39 27.94 0)
 			(show_name no)
@@
 			(project "PMM-1.0-R1"
 				(path "/dfbd1ee6-4059-4519-bc2e-4814be9dda35/f17bf38e-84eb-4b8c-8211-b5a252381cf0"
-					(reference "U6")
+					(reference "U4")
 					(unit 1)
 				)
@@
 		(dnp no)
 		(fields_autoplaced yes)
-		(property "Reference" "R17"
+		(property "Reference" "R8"
 			(at 45.72 48.2599 0)
 			(show_name no)
@@
 			(project "PMM-1.0-R1"
 				(path "/dfbd1ee6-4059-4519-bc2e-4814be9dda35/f17bf38e-84eb-4b8c-8211-b5a252381cf0"
-					(reference "R17")
-					(unit 1)
-				)
+					(reference "R8")
+					(unit 1)
+				)

Commit message: finished schematics
Parts:
- renumbered C17 to C16, C18 to C17, R9 to R10, R8 to R9, U4 to U3
Other:
- note removed: "Can it measure backward current?"
Changed lines of the file:
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@@
 	(generator_version "10.0")
 	(paper "A4")
-	(text "Can it measure backward current?"
-		(exclude_from_sim no)
-		(at 41.656 24.638 0)
-		(effects
-			(font
-				(size 1.27 1.27)
-			)
-		)
-	)
 	(junction
 		(at 43.18 45.72)
@@
 		(dnp no)
 		(fields_autoplaced yes)
-		(property "Reference" "#PWR021"
+		(property "Reference" "#PWR027"
 			(at 43.18 72.39 0)
 			(hide yes)
@@
 			(project "PMM-1.0-R1"
 				(path "/dfbd1ee6-4059-4519-bc2e-4814be9dda35/f17bf38e-84eb-4b8c-8211-b5a252381cf0"
-					(reference "#PWR021")
+					(reference "#PWR027")
 					(unit 1)
 				)
@@
 		(dnp no)
 		(fields_autoplaced yes)
-		(property "Reference" "#PWR022"
+		(property "Reference" "#PWR028"
 			(at 53.34 69.85 0)
 			(hide yes)
@@
 			(project "PMM-1.0-R1"
 				(path "/dfbd1ee6-4059-4519-bc2e-4814be9dda35/f17bf38e-84eb-4b8c-8211-b5a252381cf0"
-					(reference "#PWR022")
+					(reference "#PWR028")
 					(unit 1)
 				)
@@
 		(dnp no)
 		(fields_autoplaced yes)
-		(property "Reference" "C17"
+		(property "Reference" "C16"
 			(at 45.72 59.6962 0)
 			(show_name no)
@@
 			(project "PMM-1.0-R1"
 				(path "/dfbd1ee6-4059-4519-bc2e-4814be9dda35/f17bf38e-84eb-4b8c-8211-b5a252381cf0"
-					(reference "C17")
+					(reference "C16")
 					(unit 1)
 				)
@@
 		(dnp no)
 		(fields_autoplaced yes)
-		(property "Reference" "R9"
+		(property "Reference" "R10"
 			(at 55.88 58.4199 0)
 			(show_name no)
@@
 			(project "PMM-1.0-R1"
 				(path "/dfbd1ee6-4059-4519-bc2e-4814be9dda35/f17bf38e-84eb-4b8c-8211-b5a252381cf0"
-					(reference "R9")
+					(reference "R10")
 					(unit 1)
 				)
@@
 		(dnp no)
 		(fields_autoplaced yes)
-		(property "Reference" "#PWR023"
+		(property "Reference" "#PWR029"
 			(at 71.12 69.85 0)
 			(hide yes)
@@
 			(project "PMM-1.0-R1"
 				(path "/dfbd1ee6-4059-4519-bc2e-4814be9dda35/f17bf38e-84eb-4b8c-8211-b5a252381cf0"
-					(reference "#PWR023")
+					(reference "#PWR029")
 					(unit 1)
 				)
@@
 		(dnp no)
 		(fields_autoplaced yes)
-		(property "Reference" "C18"
+		(property "Reference" "C17"
 			(at 96.52 31.7562 0)
 			(show_name no)
@@
 			(project "PMM-1.0-R1"
 				(path "/dfbd1ee6-4059-4519-bc2e-4814be9dda35/f17bf38e-84eb-4b8c-8211-b5a252381cf0"
-					(reference "C18")
+					(reference "C17")
 					(unit 1)
 				)
@@
 		(dnp no)
 		(fields_autoplaced yes)
-		(property "Reference" "#PWR024"
+		(property "Reference" "#PWR030"
 			(at 93.98 43.18 0)
 			(hide yes)
@@
 			(project "PMM-1.0-R1"
 				(path "/dfbd1ee6-4059-4519-bc2e-4814be9dda35/f17bf38e-84eb-4b8c-8211-b5a252381cf0"
-					(reference "#PWR024")
+					(reference "#PWR030")
 					(unit 1)
 				)
@@
 		(dnp no)
 		(fields_autoplaced yes)
-		(property "Reference" "U4"
+		(property "Reference" "U3"
 			(at 72.39 27.94 0)
 			(show_name no)
@@
 			(project "PMM-1.0-R1"
 				(path "/dfbd1ee6-4059-4519-bc2e-4814be9dda35/f17bf38e-84eb-4b8c-8211-b5a252381cf0"
-					(reference "U4")
+					(reference "U3")
 					(unit 1)
 				)
@@
 		(dnp no)
 		(fields_autoplaced yes)
-		(property "Reference" "R8"
+		(property "Reference" "R9"
 			(at 45.72 48.2599 0)
 			(show_name no)
@@
 			(project "PMM-1.0-R1"
 				(path "/dfbd1ee6-4059-4519-bc2e-4814be9dda35/f17bf38e-84eb-4b8c-8211-b5a252381cf0"
-					(reference "R8")
+					(reference "R9")
 					(unit 1)
 				)

Commit message: finished schematic and started pcb routing
Parts:
- C16: footprint (none) -> Capacitor_SMD:C_0805_2012Metric
- C17: footprint (none) -> Capacitor_SMD:C_0402_1005Metric
- R10: footprint (none) -> Resistor_SMD:R_0402_1005Metric
- R9: footprint (none) -> Resistor_SMD:R_2512_6332Metric
Changed lines of the file:
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@@
 			)
 		)
-		(property "Footprint" ""
+		(property "Footprint" "Capacitor_SMD:C_0805_2012Metric"
 			(at 43.18 60.96 0)
 			(hide yes)
@@
 			)
 		)
-		(property "Footprint" ""
+		(property "Footprint" "Resistor_SMD:R_0402_1005Metric"
 			(at 53.34 59.69 0)
 			(hide yes)
@@
 			)
 		)
-		(property "Footprint" ""
+		(property "Footprint" "Capacitor_SMD:C_0402_1005Metric"
 			(at 93.98 33.02 0)
 			(hide yes)
@@
 			)
 		)
-		(property "Footprint" ""
+		(property "Footprint" "Resistor_SMD:R_2512_6332Metric"
 			(at 43.18 49.53 0)
 			(hide yes)
