File: kicad/PMM-1.0-R1.kicad_pcb (KiCad board)
At the start: 4 copper layers, 20.3 x 51.3 mm, 66 parts, among them U1 TPS61089, U2 TPS22917DBV, U3 BQ27441-G1, U4 BQ25895RTW, U5 TLV75733PDBV, U6 STM32C031C4T6

Commit message: more pcb routing
Parts:
- moved C18 27.7 mm to (38.8, 103.0), turned to 90 degrees
- moved TP1 27.1 mm to (39.1, 108.8), turned to 180 degrees
- moved C19 26.4 mm to (41.0, 103.0), turned to 90 degrees
- moved TP2 26.3 mm to (39.1, 106.2), turned to 180 degrees
- moved R19 17.9 mm to (43.0, 103.0), turned to -90 degrees
- moved C24 0.61 mm to (120.0, 150.0), turned to 90 degrees
- moved C16 0.10 mm to (16.0, 110.2)

Commit message: start routing
Parts:
- moved C3 97.2 mm to (54.8, 34.9), turned to 180 degrees
- moved C2 91.7 mm to (54.8, 37.9), turned to 180 degrees
- moved C1 86.3 mm to (54.8, 41.0), turned to 180 degrees
- moved C6 85.5 mm to (54.2, 43.6), turned to 180 degrees
- moved R6 85.0 mm to (54.2, 45.0), turned to 180 degrees
- moved R5 84.6 mm to (54.2, 46.3), turned to 0 degrees
- moved C11 82.3 mm to (55.3, 49.2), turned to -90 degrees
- moved R4 81.8 mm to (55.9, 47.6), turned to 180 degrees
- moved R2 81.3 mm to (57.3, 43.4), turned to 180 degrees
- moved C16 81.2 mm to (29.9, 30.2), turned to 180 degrees
- moved TH1 81.1 mm to (41.7, 36.6), turned to 90 degrees
- moved L1 81.0 mm to (59.6, 40.4), turned to 180 degrees
- moved C17 80.9 mm to (28.7, 28.1)
- moved R9 80.9 mm to (35.6, 30.9)
- moved U3 80.9 mm to (32.0, 27.0)
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Connections:
- net /TPS61089/TPS61089_VIN renamed /BQ25895/BQ25895_VOUT
- net BATT- renamed PACK-
- A1 pad 3: BATT+ -> PACK+
- A1 pad 4: BATT+ -> PACK+
Routing:
- net SDA: track 0.00 -> 25.8 mm, vias 0 -> 2
- net SCL: track 0.00 -> 24.9 mm, vias 0 -> 2
- net /BQ25895/BAT+: track 0.00 -> 17.9 mm
- net PACK+: track 0.00 -> 16.5 mm, vias 0 -> 2
- net Net-(U4-REGN): track 0.00 -> 14.6 mm, vias 0 -> 2
- net PACK-: track 0.00 -> 12.5 mm, vias 1 -> 9
- net Net-(U4-STAT): track 0.00 -> 8.29 mm
- net /BQ25895/BQ25895_VOUT: track 0.00 -> 8.28 mm
- net Net-(U4-TS): track 0.00 -> 7.91 mm
- net VIN: track 0.00 -> 5.59 mm
- net Net-(C20-Pad1): track 0.00 -> 4.52 mm
- net Net-(U4-ILIM): track 0.00 -> 4.38 mm
- net Net-(U4-~{QON}): track 0.00 -> 4.26 mm
- net Net-(U4-BTST): track 0.00 -> 3.90 mm
- net BQ25895_CE: track 0.00 -> 3.39 mm
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- added copper zone on F.Cu, net /BQ25895/BAT+
- added copper zone on F.Cu, net /BQ25895/BQ25895_VOUT
- added copper zone on F.Cu, net Net-(C20-Pad1)
- added copper zone on F.Cu, net PACK+
- added copper zone on In1.Cu, net PACK-

Commit message: finished pcb
Parts:
- added TP3: TestPoint, TestPoint:TestPoint_Pad_1.5x1.5mm, F.Cu at (94.3, 44.1)
- added TP4: TestPoint, TestPoint:TestPoint_Pad_1.5x1.5mm, F.Cu at (94.3, 47.6)
- moved C26 108.7 mm to (77.9, 53.4), turned to 90 degrees
- moved C25 107.2 mm to (79.6, 53.4), turned to 90 degrees
- moved U5 104.7 mm to (82.6, 53.4), turned to 180 degrees
- moved C24 102.5 mm to (85.6, 53.4), turned to -90 degrees
- moved R22 98.9 mm to (97.5, 62.6), turned to 180 degrees
- moved R21 98.4 mm to (97.5, 61.4), turned to 180 degrees
- moved R20 96.0 mm to (78.6, 57.6)
- moved U6 94.6 mm to (90.0, 62.0)
- moved D3 94.5 mm to (76.0, 56.8), turned to 90 degrees
- moved C27 91.0 mm to (83.0, 60.6), turned to 90 degrees
- moved C29 91.0 mm to (83.0, 62.6), turned to -90 degrees
- moved C28 89.8 mm to (80.6, 61.6), turned to 180 degrees
- moved R1 88.4 mm to (74.2, 53.4), turned to 90 degrees
- moved D1 87.9 mm to (76.0, 53.4), turned to 90 degrees
- moved U2 77.1 mm to (84.0, 49.0), turned to 180 degrees
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Connections:
- C15 pad 1: VOUT -> 5V_OUT
- C18 pad 1: VIN -> VBUS_5V_IN
- C19 pad 1: VIN -> VBUS_5V_IN
- R8 pad 1: VOUT -> 5V_OUT
- U2 pad 6: VOUT -> 5V_OUT
- U4 pad 1: VIN -> VBUS_5V_IN
Routing:
- net UART_TX: track 0.00 -> 51.7 mm, vias 0 -> 2
- net BQ27441_GPOUT: track 0.00 -> 50.6 mm, vias 0 -> 2
- net SCL: track 24.9 -> 73.9 mm, vias 2 -> 3
- net UART_RX: track 0.00 -> 46.4 mm, vias 0 -> 1
- net SDA: track 25.8 -> 70.5 mm, vias 2 -> 3
- net FORCE_ON: track 0.00 -> 41.1 mm, vias 0 -> 1
- net SWDIO: track 0.00 -> 40.4 mm
- net SWCLK: track 0.00 -> 38.1 mm, vias 0 -> 2
- net SHDN: track 0.00 -> 36.8 mm, vias 0 -> 1
- net +3.3V: track 3.07 -> 39.1 mm, vias 0 -> 4
- net BQ25895_CE: track 3.39 -> 34.4 mm, vias 0 -> 2
- net /TPS61089/TPS61089_VOUT: track 0.00 -> 28.3 mm, vias 1 -> 12
- net /BQ25895/BQ25895_VOUT: track 8.28 -> 36.4 mm
- net PMM_INT: track 0.00 -> 26.6 mm, vias 0 -> 1
- net BQ25895_INT: track 2.65 -> 27.7 mm, vias 0 -> 2
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- added copper zone on In2.Cu, net +3.3V
- added copper zone on B.Cu, net /TPS61089/TPS61089_VOUT
- added copper zone on F.Cu, net /TPS61089/TPS61089_VOUT
- added copper zone on F.Cu, net 5V_OUT
- added copper zone on F.Cu, net Net-(U1-SW)
- added copper zone on F.Cu, net PACK-
- added copper zone on F.Cu, net VBUS_5V_IN
- removed copper zone on F.Cu, net /BQ25895/BAT+
- removed copper zone on F.Cu, net PACK+
Other:
- board size 20.3 x 51.3 mm -> 40 x 50 mm
- board text added: "Billions must love"
- board text added: "PMM-1.0-R1"

Commit message: changes
Parts:
- moved C1 0.39 mm to (86.6, 28.2)
- moved C3 0.39 mm to (93.4, 28.2)
Routing:
- net +3.3V: track 39.1 -> 59.0 mm, vias 4 -> 6
- net ADC_IN: track 23.1 -> 24.3 mm
- net PACK-: track 36.3 -> 37.1 mm
- net SCL: track 73.9 -> 73.2 mm
- net /TPS61089/TPS61089_VOUT: vias 12 -> 11

Commit message: add stuff
Other:
- board text added: "GND GND VBAT+ VBAT+ 5V_IN 5V_IN 5V_OUT 5V_OUT 5V_OUT GND 3V3 GND SDA SCL INIT FAULT SHDN FORCE_ON PGOOD ENABLE"
- board text added: "SWDIO SWCLK NRST UART_TX UART_RX GPIO0 GPIO1 GPIO2 GPIO3 ADC_IN RESV RESV RESV RESV RESV RESV RESV RESV GND GND"

Commit message: library
Parts:
- added REF**: ESD-Logo_6.6x6mm_SilkScreen, Symbol:ESD-Logo_6.6x6mm_SilkScreen, B.Cu at (90.0, 49.5)
- added REF**: KiCad-Logo_5mm_SilkScreen, Symbol:KiCad-Logo_5mm_SilkScreen, B.Cu at (90.0, 44.7)
