File: kicad/_restore_backup_2026-07-13T18-24-17-584/PMM-1.0-R1.kicad_sch (KiCad schematic)
At the start: 3 parts

Commit message: finished schematic and started pcb routing
Parts:
- D1: footprint LED_SMD:LED_0603_1608Metric -> (none)
- R1: footprint Resistor_SMD:R_0603_1608Metric -> (none)
Other:
- note removed: "add enable r2?"
