File: kicad/_restore_backup_2026-07-13T18-24-17-584/bq25895.kicad_sch (KiCad schematic)
At the start: 21 parts, among them U4 BQ25895RTW

Commit message: finished schematic and started pcb routing
Parts:
- C18, C19: footprint Capacitor_SMD:C_0805_2012Metric -> (none)
- C20, C22, C23: footprint Capacitor_SMD:C_0603_1608Metric -> (none)
- C21: footprint Capacitor_SMD:C_0402_1005Metric -> (none)
- D2: footprint LED_SMD:LED_0603_1608Metric -> (none)
- R11, R12, R13, R14, R17, R18: footprint Resistor_SMD:R_0402_1005Metric -> (none)
- R15: footprint Resistor_SMD:R_0805_2012Metric -> (none)
- R16, R19: footprint Resistor_SMD:R_0603_1608Metric -> (none)
- TH1: value 10k NTC -> 10k 103-AT-2; footprint Resistor_SMD:R_0402_1005Metric -> (none)
- TP1, TP2: footprint TestPoint:TestPoint_Pad_1.5x1.5mm -> (none)
Changed lines of the file:
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@@
 			)
 		)
-		(property "Footprint" "Resistor_SMD:R_0603_1608Metric"
+		(property "Footprint" ""
 			(at 115.57 53.34 0)
 			(hide yes)
@@
 			)
 		)
-		(property "Footprint" "Capacitor_SMD:C_0603_1608Metric"
+		(property "Footprint" ""
 			(at 129.54 83.82 0)
 			(hide yes)
@@
 			)
 		)
-		(property "Footprint" "Capacitor_SMD:C_0603_1608Metric"
+		(property "Footprint" ""
 			(at 104.14 69.85 0)
 			(hide yes)
@@
 			)
 		)
-		(property "Footprint" "Resistor_SMD:R_0402_1005Metric"
+		(property "Footprint" ""
 			(at 58.42 91.44 0)
 			(hide yes)
@@
 			)
 		)
-		(property "Footprint" "LED_SMD:LED_0603_1608Metric"
+		(property "Footprint" ""
 			(at 106.68 36.83 0)
 			(hide yes)
@@
 			)
 		)
-		(property "Value" "10k NTC"
+		(property "Value" "10k 103-AT-2"
 			(at 132.08 112.0774 0)
 			(show_name no)
@@
 			)
 		)
-		(property "Footprint" "Resistor_SMD:R_0402_1005Metric"
+		(property "Footprint" ""
 			(at 129.54 109.22 0)
 			(hide yes)
@@
 			)
 		)
-		(property "Footprint" "Capacitor_SMD:C_0805_2012Metric"
+		(property "Footprint" ""
 			(at 50.8 58.42 0)
 			(hide yes)
@@
 			)
 		)
-		(property "Footprint" "Capacitor_SMD:C_0402_1005Metric"
+		(property "Footprint" ""
 			(at 119.38 88.9 0)
 			(hide yes)
@@
 			)
 		)
-		(property "Footprint" "Resistor_SMD:R_0402_1005Metric"
+		(property "Footprint" ""
 			(at 111.76 109.22 0)
 			(hide yes)
@@
 			)
 		)
-		(property "Footprint" "TestPoint:TestPoint_Pad_1.5x1.5mm"
+		(property "Footprint" ""
 			(at 74.93 59.69 0)
 			(hide yes)
@@
 			)
 		)
-		(property "Footprint" "Resistor_SMD:R_0603_1608Metric"
+		(property "Footprint" ""
 			(at 106.68 44.45 0)
 			(hide yes)
@@
 			)
 		)
-		(property "Footprint" "Resistor_SMD:R_0402_1005Metric"
+		(property "Footprint" ""
 			(at 111.76 101.6 0)
 			(hide yes)
@@
 			)
 		)
-		(property "Footprint" "Resistor_SMD:R_0805_2012Metric"
+		(property "Footprint" ""
 			(at 72.39 93.98 0)
 			(hide yes)
@@
 			)
 		)
-		(property "Footprint" "Resistor_SMD:R_0402_1005Metric"
+		(property "Footprint" ""
 			(at 53.34 82.55 0)
 			(hide yes)
@@
 			)
 		)
-		(property "Footprint" "Capacitor_SMD:C_0805_2012Metric"
+		(property "Footprint" ""
 			(at 60.96 58.42 0)
 			(hide yes)
@@
 			)
 		)
-		(property "Footprint" "TestPoint:TestPoint_Pad_1.5x1.5mm"
+		(property "Footprint" ""
 			(at 71.12 62.23 0)
 			(hide yes)
@@
 			)
 		)
-		(property "Footprint" "Resistor_SMD:R_0402_1005Metric"
+		(property "Footprint" ""
 			(at 34.29 71.12 0)
 			(hide yes)
@@
 			)
 		)
-		(property "Footprint" "Capacitor_SMD:C_0603_1608Metric"
+		(property "Footprint" ""
 			(at 139.7 66.04 0)
 			(hide yes)
@@
 			)
 		)
-		(property "Footprint" "Resistor_SMD:R_0402_1005Metric"
+		(property "Footprint" ""
 			(at 41.91 80.01 0)
 			(hide yes)
