File: kicad/_restore_backup_2026-07-13T18-24-17-584/stm32.kicad_sch (KiCad schematic)
At the start: 8 parts, among them U6 STM32C031C4T6

Commit message: finished schematic and started pcb routing
Parts:
- removed R21, R22: 4.7k, Resistor_SMD:R_0402_1005Metric, symbol Device:R_Small_US
- C27, C29: footprint Capacitor_SMD:C_0402_1005Metric -> (none)
- C28: footprint Capacitor_SMD:C_0603_1608Metric -> (none)
- D3: footprint LED_SMD:LED_0603_1608Metric -> (none)
- R20: footprint Resistor_SMD:R_0603_1608Metric -> (none)
