File: kicad/_restore_backup_2026-07-13T18-24-17-584/tlv75733.kicad_sch (KiCad schematic)
At the start: 4 parts, among them U5 TLV75733PDBV

Commit message: finished schematic and started pcb routing
Parts:
- C24, C25, C26: footprint Capacitor_SMD:C_0603_1608Metric -> (none)
Changed lines of the file:
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@@
 			)
 		)
-		(property "Footprint" "Capacitor_SMD:C_0603_1608Metric"
+		(property "Footprint" ""
 			(at 60.96 35.56 0)
 			(hide yes)
@@
 			)
 		)
-		(property "Footprint" "Capacitor_SMD:C_0603_1608Metric"
+		(property "Footprint" ""
 			(at 27.94 35.56 0)
 			(hide yes)
@@
 			)
 		)
-		(property "Footprint" "Capacitor_SMD:C_0603_1608Metric"
+		(property "Footprint" ""
 			(at 72.39 35.56 0)
 			(hide yes)
