File: kicad/_restore_backup_2026-07-13T18-24-17-584/tps22917.kicad_sch (KiCad schematic)
At the start: 7 parts, among them U2 TPS22917DBV

Commit message: finished schematic and started pcb routing
Parts:
- C12, C13, C15: footprint Capacitor_SMD:C_0805_2012Metric -> (none)
- C14: footprint Capacitor_SMD:C_0402_1005Metric -> (none)
- R7: footprint Resistor_SMD:R_0402_1005Metric -> (none)
- R8: footprint Resistor_SMD:R_0603_1608Metric -> (none)
Changed lines of the file:
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@@
 			)
 		)
-		(property "Footprint" "Capacitor_SMD:C_0805_2012Metric"
+		(property "Footprint" ""
 			(at 36.83 44.45 0)
 			(hide yes)
@@
 			)
 		)
-		(property "Footprint" "Capacitor_SMD:C_0805_2012Metric"
+		(property "Footprint" ""
 			(at 25.4 44.45 0)
 			(hide yes)
@@
 			)
 		)
-		(property "Footprint" "Capacitor_SMD:C_0402_1005Metric"
+		(property "Footprint" ""
 			(at 46.99 43.18 0)
 			(hide yes)
@@
 			)
 		)
-		(property "Footprint" "Resistor_SMD:R_0603_1608Metric"
+		(property "Footprint" ""
 			(at 81.28 44.45 0)
 			(hide yes)
@@
 			)
 		)
-		(property "Footprint" "Resistor_SMD:R_0402_1005Metric"
+		(property "Footprint" ""
 			(at 55.88 53.34 0)
 			(hide yes)
@@
 			)
 		)
-		(property "Footprint" "Capacitor_SMD:C_0805_2012Metric"
+		(property "Footprint" ""
 			(at 91.44 44.45 0)
 			(hide yes)
