File: kicad/_restore_backup_2026-07-13T18-24-17-584/tps61089.kicad_sch (KiCad schematic)
At the start: 18 parts, among them U1 TPS61089

Commit message: finished schematic and started pcb routing
Parts:
- C1, C10, C2, C3, C8: footprint Capacitor_SMD:C_1210_3225Metric -> (none)
- C11, C4, C7, C9: footprint Capacitor_SMD:C_0402_1005Metric -> (none)
- C5: footprint Capacitor_SMD:C_0805_2012Metric -> (none)
- C6: footprint Capacitor_SMD:C_0603_1608Metric -> (none)
- L1: value 470nH Coilcraft XFL4015-471MEC -> 470nH; footprint Inductor_SMD:L_Coilcraft_XxL4020 -> (none)
- R2, R3, R4, R6: footprint Resistor_SMD:R_0402_1005Metric -> (none)
- R5: footprint Resistor_SMD:R_0603_1608Metric -> (none)
Changed lines of the file:
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@@
-		)
-	)
-	(label "TPS61089_VOUT"
-		(at 115.57 36.83 0)
-		(effects
-			(font
-				(size 1.27 1.27)
-			)
-			(justify left bottom)
-		)
-	)
-	(label "TPS61089_VIN"
-		(at 36.83 45.72 0)
-		(effects
-			(font
-				(size 1.27 1.27)
-			)
-			(justify left bottom)
 		)
 	)
@@
 			)
 		)
-		(property "Footprint" "Capacitor_SMD:C_0402_1005Metric"
+		(property "Footprint" ""
 			(at 115.57 40.64 0)
 			(hide yes)
@@
 			)
 		)
-		(property "Footprint" "Capacitor_SMD:C_0402_1005Metric"
+		(property "Footprint" ""
 			(at 133.35 62.23 0)
 			(hide yes)
@@
 			)
 		)
-		(property "Footprint" "Capacitor_SMD:C_1210_3225Metric"
+		(property "Footprint" ""
 			(at 127 40.64 0)
 			(hide yes)
@@
 			)
 		)
-		(property "Value" "470nH Coilcraft XFL4015-471MEC"
+		(property "Value" "470nH"
 			(at 69.85 41.91 90)
 			(show_name no)
@@
 			)
 		)
-		(property "Footprint" "Inductor_SMD:L_Coilcraft_XxL4020"
+		(property "Footprint" ""
 			(at 69.85 45.72 0)
 			(hide yes)
@@
 			)
 		)
-		(property "Footprint" "Capacitor_SMD:C_0603_1608Metric"
+		(property "Footprint" ""
 			(at 113.03 64.77 0)
 			(hide yes)
@@
 			)
 		)
-		(property "Footprint" "Capacitor_SMD:C_1210_3225Metric"
+		(property "Footprint" ""
 			(at 36.83 49.53 0)
 			(hide yes)
@@
 			)
 		)
-		(property "Footprint" "Resistor_SMD:R_0402_1005Metric"
+		(property "Footprint" ""
 			(at 142.24 59.69 0)
 			(hide yes)
@@
 			)
 		)
-		(property "Footprint" "Resistor_SMD:R_0402_1005Metric"
+		(property "Footprint" ""
 			(at 73.66 49.53 0)
 			(hide yes)
@@
 			)
 		)
-		(property "Footprint" "Resistor_SMD:R_0402_1005Metric"
+		(property "Footprint" ""
 			(at 158.75 54.61 0)
 			(hide yes)
@@
 			)
 		)
-		(property "Footprint" "Resistor_SMD:R_0402_1005Metric"
+		(property "Footprint" ""
 			(at 124.46 64.77 0)
 			(hide yes)
@@
 			)
 		)
-		(property "Footprint" "Capacitor_SMD:C_0805_2012Metric"
+		(property "Footprint" ""
 			(at 83.82 49.53 0)
 			(hide yes)
@@
 			)
 		)
-		(property "Footprint" "Resistor_SMD:R_0603_1608Metric"
+		(property "Footprint" ""
 			(at 158.75 46.99 0)
 			(hide yes)
@@
 			)
 		)
-		(property "Footprint" "Capacitor_SMD:C_0402_1005Metric"
+		(property "Footprint" ""
 			(at 142.24 66.04 0)
 			(hide yes)
@@
 			)
 		)
-		(property "Footprint" "Capacitor_SMD:C_0402_1005Metric"
+		(property "Footprint" ""
 			(at 57.15 49.53 0)
 			(hide yes)
@@
 			)
 		)
-		(property "Footprint" "Capacitor_SMD:C_1210_3225Metric"
+		(property "Footprint" ""
 			(at 137.16 40.64 0)
 			(hide yes)
@@
 			)
 		)
-		(property "Footprint" "Capacitor_SMD:C_1210_3225Metric"
+		(property "Footprint" ""
 			(at 26.67 49.53 0)
 			(hide yes)
@@
 			)
 		)
-		(property "Footprint" "Capacitor_SMD:C_1210_3225Metric"
+		(property "Footprint" ""
 			(at 46.99 49.53 0)
 			(hide yes)
