File: kicad/_restore_backup_2026-07-17T16-44-49-099/PMM-1.0-R1.kicad_pcb (KiCad board)
At the start: 4 copper layers, 40 x 50 mm, 74 parts, among them U1 TPS61089, U2 TPS22917DBV, U3 BQ27441-G1, U4 BQ25895RTW, U5 TLV75733PDBV, U6 STM32C031C4T6

Commit message: add silkscreen
Other:
- board text added: "GND GND VBAT+ VBAT+ 5V_IN 5V_IN 5V_OUT 5V_OUT 5V_OUT GND 3V3 GND SDA SCL INIT FAULT SHDN FORCE_ON PGOOD ENABLE"
- board text removed: "DATE:"
- board text removed: "GND GND VBAT+ VBAT+ 5V_IN 5V_IN 5V_OUT 5V_OUT 5V_OUT GND 3V3 GND SDA SCL INIT FAULT SHDN FORCE PGOOD ENABLE"
- board text removed: "TEST:"
- board text removed: ""
Changed lines of the file:
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@@
 		)
 	)
-	(gr_text ""
-		(at 98.9 77.4 0)
-		(layer "B.SilkS")
-		(effects
-			(font
-				(size 1 1)
-				(thickness 0.1)
-			)
-			(justify left bottom mirror)
-		)
-	)
 	(gr_text "SWDIO\nSWCLK\nNRST\nUART_TX\nUART_RX\nGPIO0\nGPIO1\nGPIO2\nGPIO3\nADC_IN\nRESV\nRESV\nRESV\nRESV\nRESV\nRESV\nRESV\nRESV\nGND\nGND"
 		(at 107 75 0)
@@
 		)
 	)
-	(gr_text "GND\nGND\nVBAT+\nVBAT+\n5V_IN\n5V_IN\n5V_OUT\n5V_OUT\n5V_OUT\nGND\n3V3\nGND\nSDA\nSCL\nINIT\nFAULT\nSHDN\nFORCE\nPGOOD\nENABLE"
+	(gr_text "GND\nGND\nVBAT+\nVBAT+\n5V_IN\n5V_IN\n5V_OUT\n5V_OUT\n5V_OUT\nGND\n3V3\nGND\nSDA\nSCL\nINIT\nFAULT\nSHDN\nFORCE_ON\nPGOOD\nENABLE"
 		(at 73 75 0)
 		(layer "B.SilkS")
@@
 		)
 	)
-	(gr_text "TEST:"
-		(at 93.7 68 0)
-		(layer "B.SilkS" knockout)
-		(effects
-			(font
-				(face "JetBrainsMono NFM")
-				(size 1 1)
-				(thickness 0.1)
-			)
-			(justify mirror)
-		)
-		(render_cache "TEST:" 0
-			(polygon
-				(pts
-					(xy 95.441268 68.415) (xy 95.441268 67.508431) (xy 95.721109 67.508431) (xy 95.721109 67.393698)
-					(xy 95.03558 67.393698) (xy 95.03558 67.508431) (xy 95.315361 67.508431) (xy 95.315361 68.415)
-				)
-			)
-			(polygon
-				(pts
-					(xy 94.818937 68.415) (xy 94.818937 67.393698) (xy 94.23135 67.393698) (xy 94.23135 67.508431)
-					(xy 94.694434 67.508431) (xy 94.694434 67.824603) (xy 94.28032 67.824603) (xy 94.28032 67.936528)
-					(xy 94.694434 67.936528) (xy 94.694434 68.300266) (xy 94.23135 68.300266) (xy 94.23135 68.415)
-				)
-			)
-			(polygon
-				(pts
-					(xy 93.694321 68.428982) (xy 93.768186 68.423558) (xy 93.831043 68.40822) (xy 93.884745 68.38386)
-					(xy 93.930748 68.350642) (xy 93.968697 68.30864) (xy 93.99595 68.259742) (xy 94.012893 68.20258)
-					(xy 94.018858 68.135219) (xy 93.892951 68.135219) (xy 93.886469 68.189642) (xy 93.868211 68.233348)
-					(xy 93.838424 68.26882) (xy 93.799491 68.294962) (xy 93.752203 68.311257) (xy 93.694321 68.317058)
-					(xy 93.638506 68.311035) (xy 93.593108 68.294081) (xy 93.555835 68.266683) (xy 93.527391 68.23025)
-					(xy 93.510111 68.187088) (xy 93.504056 68.135219) (xy 93.507855 68.095222) (xy 93.51886 68.059855)
-					(xy 93.536967 68.02818) (xy 93.561565 68.00146) (xy 93.592625 67.98074) (xy 93.631367 67.965898)
-					(xy 93.786645 67.922545) (xy 93.847557 67.898411) (xy 93.897627 67.865154) (xy 93.938442 67.822527)
-					(xy 93.968926 67.772087) (xy 93.987356 67.715941) (xy 93.993701 67.652534) (xy 93.989465 67.599438)
-					(xy 93.977229 67.552213) (xy 93.957309 67.509836) (xy 93.929886 67.471943) (xy 93.896083 67.440151)
-					(xy 93.855216 67.414031) (xy 93.810214 67.395291) (xy 93.760155 67.383724) (xy 93.704091 67.379715)
-					(xy 93.647119 67.383734) (xy 93.596398 67.395311) (xy 93.55095 67.414031) (xy 93.509445 67.440107)
-					(xy 93.47493 67.471693) (xy 93.44672 67.509164) (xy 93.425975 67.551139) (xy 93.413298 67.597653)
-					(xy 93.408923 67.649726) (xy 93.53483 67.649726) (xy 93.540322 67.605195) (xy 93.556111 67.567753)
-					(xy 93.582397 67.535725) (xy 93.616396 67.51158) (xy 93.656403 67.496817) (xy 93.704091 67.491639)
-					(xy 93.751746 67.496846) (xy 93.791269 67.511629) (xy 93.824441 67.535725) (xy 93.84989 67.567649)
-					(xy 93.865247 67.605095) (xy 93.870603 67.649726) (xy 93.867103 67.686039) (xy 93.857019 67.717679)
-					(xy 93.8405 67.745591) (xy 93.818157 67.769086) (xy 93.790281 67.787477) (xy 93.75587 67.800851)
-					(xy 93.596379 67.845608) (xy 93.532145 67.870385) (xy 93.479811 67.905481) (xy 93.437561 67.951243)
-					(xy 93.406418 68.005402) (xy 93.387455 68.066171) (xy 93.380896 68.135219) (xy 93.386642 68.201219)
-					(xy 93.40302 68.257801) (xy 93.429439 68.306721) (xy 93.466259 68.349237) (xy 93.511048 68.383234)
-					(xy 93.563008 68.407999) (xy 93.623505 68.423512)
-				)
-			)
-			(polygon
-				(pts
-					(xy 92.923612 68.415) (xy 92.923612 67.508431) (xy 93.203454 67.508431) (xy 93.203454 67.393698)
-					(xy 92.517925 67.393698) (xy 92.517925 67.508431) (xy 92.797705 67.508431) (xy 92.797705 68.415)
-				)
-			)
-			(polygon
-				(pts
-					(xy 92.02144 67.838586) (xy 92.05871 67.835052) (xy 92.086932 67.82546) (xy 92.108208 67.810621)
-					(xy 92.124243 67.790291) (xy 92.13409 67.765545) (xy 92.137578 67.735088) (xy 92.13409 67.704632)
-					(xy 92.124243 67.679886) (xy 92.108208 67.659556) (xy 92.086927 67.644682) (xy 92.058705 67.635071)
-					(xy 92.02144 67.63153) (xy 91.984218 67.63507) (xy 91.956014 67.64468) (xy 91.934734 67.659556)
-					(xy 91.918699 67.679886) (xy 91.908852 67.704632) (xy 91.905364 67.735088) (xy 91.908852 67.765545)
-					(xy 91.918699 67.790291) (xy 91.934734 67.810621) (xy 91.956009 67.825462) (xy 91.984213 67.835053)
-				)
-			)
-			(polygon
-				(pts
-					(xy 92.02144 68.428982) (xy 92.05871 68.425448) (xy 92.086932 68.415856) (xy 92.108208 68.401017)
-					(xy 92.124243 68.380687) (xy 92.13409 68.355941) (xy 92.137578 68.325484) (xy 92.13409 68.295028)
-					(xy 92.124243 68.270282) (xy 92.108208 68.249952) (xy 92.086927 68.235078) (xy 92.058705 68.225467)
-					(xy 92.02144 68.221926) (xy 91.984218 68.225466) (xy 91.956014 68.235076) (xy 91.934734 68.249952)
-					(xy 91.918699 68.270282) (xy 91.908852 68.295028) (xy 91.905364 68.325484) (xy 91.908852 68.355941)
-					(xy 91.918699 68.380687) (xy 91.934734 68.401017) (xy 91.956009 68.415858) (xy 91.984213 68.425449)
-				)
-			)
-		)
-	)
-	(gr_text "DATE:"
-		(at 93.7 69.4 0)
-		(layer "B.SilkS" knockout)
-		(effects
-			(font
-				(face "JetBrainsMono NFM")
-				(size 1 1)
-				(thickness 0.1)
-			)
-			(justify mirror)
-		)
-		(render_cache "DATE:" 0
-			(polygon
-				(pts
-					(xy 95.66933 69.815) (xy 95.404937 69.815) (xy 95.339589 69.810501) (xy 95.282912 69.797698) (xy 95.233539 69.777264)
-					(xy 95.18884 69.748383) (xy 95.151769 69.712889) (xy 95.121615 69.670225) (xy 95.099891 69.622544)
-					(xy 95.086434 69.568618) (xy 95.081742 69.507192) (xy 95.081742 69.100101) (xy 95.207649 69.100101)
-					(xy 95.207649 69.507192) (xy 95.214023 69.566635) (xy 95.23177 69.613766) (xy 95.260162 69.651357)
-					(xy 95.2981 69.679315) (xy 95.345459 69.696801) (xy 95.404937 69.703075) (xy 95.543422 69.703075)
-					(xy 95.543422 68.905622) (xy 95.404937 68.905622) (xy 95.345464 68.911903) (xy 95.298104 68.929408)
-					(xy 95.260162 68.957402) (xy 95.231703 68.994961) (xy 95.213988 69.041648) (xy 95.207649 69.100101)
-					(xy 95.081742 69.100101) (xy 95.086447 69.03868) (xy 95.099914 68.985015) (xy 95.121615 68.937801)
-					(xy 95.151729 68.895563) (xy 95.188795 68.860302) (xy 95.233539 68.831495) (xy 95.282915 68.811027)
-					(xy 95.339593 68.798203) (xy 95.404937 68.793698) (xy 95.66933 68.793698)
-				)
-			)
-			(polygon
-				(pts
-					(xy 94.888852 69.815) (xy 94.760136 69.815) (xy 94.69303 69.543585) (xy 94.383818 69.543585) (xy 94.316652 69.815)
-					(xy 94.18934 69.815) (xy 94.287147 69.437278) (xy 94.41038 69.437278) (xy 94.667812 69.437278)
-					(xy 94.589471 69.121106) (xy 94.554544 68.972789) (xy 94.539096 68.894448) (xy 94.52377 68.972789)
-					(xy 94.488782 69.12251) (xy 94.41038 69.437278) (xy 94.287147 69.437278) (xy 94.453794 68.793698)
-					(xy 94.623054 68.793698)
-				)
-			)
-			(polygon
-				(pts
-					(xy 93.762831 69.815) (xy 93.762831 68.908431) (xy 94.042672 68.908431) (xy 94.042672 68.793698)
-					(xy 93.357144 68.793698) (xy 93.357144 68.908431) (xy 93.636924 68.908431) (xy 93.636924 69.815)
-				)
-			)
-			(polygon
-				(pts
-					(xy 93.1405 69.815) (xy 93.1405 68.793698) (xy 92.552913 68.793698) (xy 92.552913 68.908431) (xy 93.015997 68.908431)
-					(xy 93.015997 69.224603) (xy 92.601884 69.224603) (xy 92.601884 69.336528) (xy 93.015997 69.336528)
-					(xy 93.015997 69.700266) (xy 92.552913 69.700266) (xy 92.552913 69.815)
-				)
-			)
-			(polygon
-				(pts
-					(xy 92.02144 69.238586) (xy 92.05871 69.235052) (xy 92.086932 69.22546) (xy 92.108208 69.210621)
-					(xy 92.124243 69.190291) (xy 92.13409 69.165545) (xy 92.137578 69.135088) (xy 92.13409 69.104632)
-					(xy 92.124243 69.079886) (xy 92.108208 69.059556) (xy 92.086927 69.044682) (xy 92.058705 69.035071)
-					(xy 92.02144 69.03153) (xy 91.984218 69.03507) (xy 91.956014 69.04468) (xy 91.934734 69.059556)
-					(xy 91.918699 69.079886) (xy 91.908852 69.104632) (xy 91.905364 69.135088) (xy 91.908852 69.165545)
-					(xy 91.918699 69.190291) (xy 91.934734 69.210621) (xy 91.956009 69.225462) (xy 91.984213 69.235053)
-				)
-			)
-			(polygon
-				(pts
-					(xy 92.02144 69.828982) (xy 92.05871 69.825448) (xy 92.086932 69.815856) (xy 92.108208 69.801017)
-					(xy 92.124243 69.780687) (xy 92.13409 69.755941) (xy 92.137578 69.725484) (xy 92.13409 69.695028)
-					(xy 92.124243 69.670282) (xy 92.108208 69.649952) (xy 92.086927 69.635078) (xy 92.058705 69.625467)
-					(xy 92.02144 69.621926) (xy 91.984218 69.625466) (xy 91.956014 69.635076) (xy 91.934734 69.649952)
-					(xy 91.918699 69.670282) (xy 91.908852 69.695028) (xy 91.905364 69.725484) (xy 91.908852 69.755941)
-					(xy 91.918699 69.780687) (xy 91.934734 69.801017) (xy 91.956009 69.815858) (xy 91.984213 69.825449)
-				)
-			)
-		)
-	)
 	(gr_text "SN:"
 		(at 94.6 66.6 0)
@@
 			)
 		)
-	)
-	(zone
-		(layer "B.SilkS")
-		(hatch edge 0.5)
-		(connect_pads yes
-			(clearance 0.5)
-		)
-		(min_thickness 0.25)
-		(fill yes
-			(thermal_gap 0.5)
-			(thermal_bridge_width 0.5)
-			(island_removal_mode 0)
-		)
-		(polygon
-			(pts
-				(xy 91.7 68.7) (xy 91.7 69.9) (xy 84.1 69.9) (xy 84.1 68.7)
-			)
-		)
-	)
-	(zone
-		(layer "B.SilkS")
-		(hatch edge 0.5)
-		(connect_pads yes
-			(clearance 0.5)
-		)
-		(min_thickness 0.25)
-		(fill yes
-			(thermal_gap 0.5)
-			(thermal_bridge_width 0.5)
-			(island_removal_mode 0)
-		)
-		(polygon
-			(pts
-				(xy 91.7 67.300123) (xy 91.7 68.500123) (xy 84.1 68.500123) (xy 84.1 67.300123)
-			)
-		)
